File: DaughterBoard1.0/DaughterBoard1.0.kicad_sch (KiCad schematic)
At the start: 71 parts, among them J1 VP0265540000G, J10 B3B-EH-ALFSN, J11 B3B-EH-ALFSN, J12 B3B-EH-ALFSN, J13 25SH-C-04-TS, J15 25SH-C-04-TS, J16 25SH-C-04-TS, J17 25SH-C-04-TS, J18 440052-5, J19 440052-5, J2 1744057-6, J20 B3B-EH-ALFSN, J21 25SH-C-04-TS, J22 25SH-C-04-TS, J23 1-1123723-5, J24 68000-103HLF, J25 B3B-EH-ALFSN, J26 68000-103HLF, J27 61300211121, J28 61300211121, J29 61300211121, J3 1744057-6, J30 61300211121, J31 61300211121, J32 61300211121, J33 61300211121, J34 61300211121, J35 61300211121, J36 61300211121, J37 61300211121, J38 61300211121, J39 61300211121, J4 1744057-6, J40 61300211121, J41 61300211121, J42 61300211121, J43 61300211121, J44 61300211121, J45 1-1123723-4, J46 B3B-EH-ALFSN, J47 B3B-EH-ALFSN, J48 B3B-EH-ALFSN, J49 B3B-EH-ALFSN, J5 1744057-6, J50 B3B-EH-ALFSN, J51 61300211121, J52 61300211121, J53 61300211121, J54 61300211121, J55 61300211121, J6 1744057-6, J7 1744057-6, J8 RS2-14-G, J9 B3B-EH-ALFSN, U1 ATMEGA2560-16AUR, U2 PTS636, U4 ADG804YRMZ

Commit message: Updated version, basically complete. Will keep better updates moving forward
Parts:
- removed J10, J50, J9: B3B-EH-ALFSN, ServoHeader:CONN3_B3B-EH-ALFSN_JST, symbol ServoHeader:B3B-EH-ALFSN
- removed J22: 25SH-C-04-TS, 4PinHeader:CONN_B4B-EH-A_JST, symbol 4PinHeader:B4B-EH-ALFSN
- removed J45: 1-1123723-4, 4PinHeader7.5A:TE_1-1123723-4, symbol 4PinHeader7.5A:1-1123723-4
- removed J55: 61300211121, 2PinDupont:CONN_61300211121_WRE, symbol 2PinDupont:61300211121
- added C10, C11, C12, C13, C14, C9: DNP, Capacitor_SMD:C_0603_1608Metric, symbol Device:C
- added C15, C16: 0.1uF, Capacitor_SMD:C_0603_1608Metric, symbol Device:C
- added C18: 0.1uF, Capacitor_SMD:C_0805_2012Metric_Pad1.18x1.45mm_HandSolder, symbol Device:C
- added C19: TAJC226M016RNJ, BigCapacitor:TAJC_AVX, symbol BigCap:TAJC226M016RNJ
- added G1: LOGO, Logo:logo, symbol Logo:LOGO
- added J10, J57, J58, J59, J60, J61, J62, J63, J64, J65, J66, J67, J9: 61300211121, 2PinDupont:CONN_61300211121_WRE, symbol 2PinDupont:61300211121
- added J17: 25SH-C-04-TS, 4PinHeader:CONN_B4B-EH-A_JST, symbol 4PinHeader:B4B-EH-ALFSN
- added J22, J50, J55: 691137710002, CONN2_710002_WRE, symbol LEDScrewTerm:691137710002
- added J45: B3B-EH-ALFSN, ServoHeader:CONN3_B3B-EH-ALFSN_JST, symbol ServoHeader:B3B-EH-ALFSN
- added J56: 440052-5, 5PinHeader7.5A:conn5_1-1123723-5_TEC, symbol 5PinHeader:440052-5
- added Q1, Q2, Q3: G35N02K, HeadlightFet:QNMOS1G2D3S_TO252DPAK_DIO, symbol HeadlightFet:DMN10H170SK3-13
- added R7: 1K, Resistor_SMD:R_0603_1608Metric, symbol Device:R_US
- added R8: 6.9K, Resistor_SMD:R_0603_1608Metric, symbol Device:R_US
- added R9: LTO050FR0100JTE3, TO220_LTO_VIS, symbol ShuntResistor:LTO050FR0100JTE3
- added U3: MCP9700T-E/TT, SOT-23_MC_MCH, symbol TempSensor:MCP9700T-E_TT
- added U5: LT6106CS5-TRMPBF, TSOT-23-5_S5_ADI, symbol CurrentSense:LT6106CS5-TRMPBF
- added U8: BA90DD0WHFP-TR, LDO:HRP5_ROM, symbol LDO:BA90DD0WHFP-TR
- renumbered J15 to J14, J16 to J15, J17 to J16, J4 to J3, J6 to J4, J3 to J5, J5 to J6
Connections:
- net 12V: now also C13.1, C14.1, C18.1, J22.2, J50.2, J55.2, J56.1, R7.1, R9.2, U5.5 (V+), U8.1 (CTL), U8.2 (Vcc); no longer J1.1, J1.2, J19.1
- net 3V3: now also C10.1, C9.1
- net 5V: now also C11.1, C12.1, C15.1, J17.1, J45.1, U3.1 (VDD)
- net ADC1: now also J3.3; no longer J5.3
- net ADC10: now also J51.2; no longer J53.1
- net ADC11: now also J52.1; no longer J53.2
- net ADC12: now also J52.2; no longer J54.1
- net ADC13: now also J53.1; no longer J54.2
- net ADC14: now also J53.2
- net ADC15: now also J54.1
- net ADC2: now also J4.3; no longer J3.3
- net ADC3: now also J5.3; no longer J6.3
- net ADC4: now also J6.3; no longer J4.3
- net ADC6: now also U3.2 (VOUT); no longer J51.1
- net ADC7: now also J45.3; no longer J51.2
- net ADC8: now also R8.1, U5.1 (OUT); no longer J52.1
- net ADC9: now also J51.1; no longer J52.2
- net GND: now also C10.2, C11.2, C12.2, C13.2, C14.2, C15.2, C16.2, C18.2, C19.2, C9.2, J17.2, J45.2, J56.2, Q1.3 (S), Q2.3 (S), Q3.3 (S), R8.2, U3.3 (GND), U5.2 (V-), U8.3 (GND), U8.6 (EPAD)
- net I2C_SCL: now also J17.4, J56.4
- net I2C_SDA: now also J17.3, J56.3
- net Motor1 brake: now also U1.9 (PE7(CLKO/ICP3/INT7)); no longer U1.8 (PE6(T3/INT6))
- net Motor2 brake: now also J3.6; no longer J5.6
- net Motor2 dir: now also J3.4, U1.8 (PE6(T3/INT6)); no longer J5.4, U1.9 (PE7(CLKO/ICP3/INT7))
- net Motor3 brake: now also J4.6, U1.37 (PL2(T5)); no longer J3.6, U1.35 (PL0(ICP4))
- net Motor3 dir: now also J4.4, U1.36 (PL1(ICP5)); no longer J3.4, U1.27 (PH7(T4))
- net Motor4 brake: now also J5.6, U1.35 (PL0(ICP4)); no longer J6.6, U1.37 (PL2(T5))
- net Motor4 dir: now also J5.4, U1.27 (PH7(T4)); no longer J6.4, U1.36 (PL1(ICP5))
- net Motor5 brake: now also J6.6; no longer J4.6
- net Motor5 dir: now also J6.4; no longer J4.4
- net PWM Timer0 B: now also Q1.1 (G)
- net PWM Timer2 A: now also Q3.1 (G)
- net PWM Timer2 B: now also Q2.1 (G)
- net PWM Timer3 B: now also J3.5; no longer J5.5
- net PWM Timer3 C: now also J4.5; no longer J3.5
- net PWM Timer4 A: now also J5.5; no longer J6.5
- net PWM Timer4 B: now also J6.5; no longer J4.5
- net Thermal camera: now reaches J21.3, U4.4 (S3)
- net Ext1: now reaches U1.19 (PB0(*SS/PCINT0))
- net Ext1: now also J9.1
- net Ext2: now reaches U1.28 (PG3(TOSC2))
- net Ext2: now also J9.2
- net Ext3: now reaches U1.29 (PG4(TOSC1))
- net Ext3: now also J10.1
- net Ext26: now reaches U1.51 (PG0(*WR))
- net Ext26: now also J67.2
- net Ext25: now reaches U1.52 (PG1(*RD))
- net Ext25: now also J67.1
- net Ext23: now reaches U1.56 (PC3(A11))
- net Ext23: now also J66.1
- net Ext22: now reaches U1.57 (PC4(A12))
- net Ext22: now also J65.2
- net Ext21: now reaches U1.58 (PC5(A13))
- net Ext21: now also J65.1
- net Ext20: now reaches U1.59 (PC6(A14))
- net Ext20: now also J64.2
- net Ext19: now reaches U1.60 (PC7(A15))
- net Ext19: now also J64.1
- net Ext18: now reaches U1.65 (PJ2(XCK3/PCINT11))
- net Ext18: now also J63.2
- net Ext17: now reaches U1.66 (PJ3(PCINT12))
- net Ext17: now also J63.1
- net Ext16: now reaches U1.67 (PJ4(PCINT13))
- net Ext16: now also J62.2
- net Ext15: now reaches U1.68 (PJ5(PCINT14))
- net Ext15: now also J62.1
- net Ext14: now reaches U1.69 (PJ6(PCINT15))
- net Ext14: now also J61.2
- net Ext13: now reaches U1.70 (PG2(ALE))
- net Ext13: now also J61.1
- net Ext12: now reaches U1.71 (PA7(AD7))
- net Ext12: now also J60.2
- net Ext11: now reaches U1.72 (PA6(AD6))
- net Ext11: now also J60.1
- net Ext10: now reaches U1.73 (PA5(AD5))
- net Ext10: now also J59.2
- net Ext9: now reaches U1.74 (PA4(AD4))
- net Ext9: now also J59.1
- net Ext8: now reaches U1.75 (PA3(AD3))
- net Ext8: now also J58.2
- net Ext7: now reaches U1.76 (PA2(AD2))
- net Ext7: now also J58.1
- net Ext6: now reaches U1.77 (PA1(AD1))
- net Ext6: now also J57.2
- net Ext5: now reaches U1.78 (PA0(AD0))
- net Ext5: now also J57.1
- net Ext4: now reaches U1.79 (PJ7)
- net Ext4: now also J10.2
- net at U1.98 (AREF): now also C16.1
- net Auxilary camera: now reaches U4.7 (S4)
- net Auxilary camera: now also J56.5
- net Auxilary control renamed Ext24
- net Ext24: now also J66.2
- new net: J1.1, J1.2, R9.1, U5.4 (+IN)
- new net: J55.1, Q3.2 (D)
- new net: R7.2, U5.3 (-IN)
- new net: C19.1, J19.1, U8.4 (OUT)
- new net: J22.1, Q1.2 (D)
- new net: J50.1, Q2.2 (D)
Other:
- note added: "Current Sensing"
- note added: "Extra Pins"
- note added: "I2C Headers"
- note added: "LED Headlight Drivers"
- note added: "Noise Suppression Caps"
- note added: "SM Temperature Sensor"
- note added: "Temperature Sensor Header"
- note removed: "Auxiliary Camera"
- note removed: "I2C Header"
- moved on the sheet: C1, C2, C3, C4, C5, C6, C7, C8, J1, J11, J12, J13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
